Commit message: Rename repo my_SOARM100, describe arm in URDF, update notes
- rename repo to `my_SOARM100`

- in `.gitignore` -> add
  `raw_videos` for heavy raw video material,
  `secrets.txt` for secrets,
  `__pycache__` for temp python files

- in `URDF.md` -> complete notes to model robotic arm in URDF from scratch,
  update references to new repo name: `my_SOARM100`

- in folder `src/my_arm_description`:
  - rename `/meshes/Moving Jaw.STL`to `Moving_Jaw.STL`
  - in `/meshes/my_arm.FCStd` -> finish model of the robotic arm in FreeCAD
  - in `/urdf/my_arm.urdf.xacro` -> finish model of the robotic arm in URDF

File: src/my_arm_description/urdf/my_arm.urdf.xacro (robot description, xacro)
@@ -4,5 +4,5 @@
     <link name="base_link">
         <visual>
-            <origin xyz="-0.0452 0 0" rpy="0 0 ${pi/2}" />
+            <origin xyz="0.0 0.0 0.0" rpy="0 0 0" />
             <geometry>
                 <mesh filename="package://my_arm_description/meshes/Base.STL" />
@@ -10,5 +10,5 @@
         </visual>
     </link>
-    <joint name="world_to_base" type="fixed">
+    <joint name="world_to_base_joint" type="fixed">
         <origin xyz="0.0 0.0 0.0" rpy="0 0 0" />
         <parent link="world" />
@@ -17,5 +17,5 @@
     <link name="shoulder_link">
         <visual>
-            <origin xyz="0 0 0.0165" rpy="${pi/2} 0 ${pi/2}" />
+            <origin xyz="0 0 0" rpy="${pi/2} 0 0" />
             <geometry>
                 <mesh filename="package://my_arm_description/meshes/Rotation_Pitch.STL" />
@@ -23,12 +23,14 @@
         </visual>
     </link>
-    <joint name="base_to_shoulder" type="rotation">
-        <origin xyz="0.0 0.0 0.0" rpy="0 0 ${0}" />
+    <joint name="base_to_shoulder_joint" type="revolute">
+        <origin xyz="0 -0.0452 0.0165" rpy="0 0 0" />
         <parent link="base_link" />
         <child link="shoulder_link" />
+        <axis xyz="0 0 1" />
+        <limit upper="${pi/2}" lower="-${pi/2}" effort="1.0" velocity="1.0" />
     </joint>
     <link name="upper_arm_link">
         <visual>
-            <origin xyz="0 0 0" rpy="${pi/2} 0 ${pi/2}" />
+            <origin xyz="0 0 0" rpy="0 ${pi/2} 0" />
             <geometry>
                 <mesh filename="package://my_arm_description/meshes/Upper_Arm.STL" />
@@ -36,8 +38,70 @@
         </visual>
     </link>
-    <joint name="shoulder_to_upper_arm" type="rotation">
-        <origin xyz="0.0306 0.0 0.1190 " rpy="0 0 0" />
+    <joint name="shoulder_to_upper_arm_joint" type="revolute">
+        <origin xyz="0 -0.0306 0.10 " rpy="${pi/2} 0 -${pi/2}" />
         <parent link="shoulder_link" />
         <child link="upper_arm_link" />
+        <axis xyz="0 0 1" />
+        <limit upper="${pi/2}" lower="-${pi/2}" effort="1.0" velocity="1.0" />
+    </joint>
+    <link name="lower_arm_link">
+        <visual>
+            <origin xyz="0 0 0" rpy="0 ${pi/2} 0" />
+            <geometry>
+                <mesh filename="package://my_arm_description/meshes/Lower_Arm.STL" />
+            </geometry>
+        </visual>
+    </link>
+    <joint name="upper_arm_to_lower_arm_joint" type="revolute">
+        <origin xyz="0.0276 0.1125 0.0" rpy="0 0 0" />
+        <parent link="upper_arm_link" />
+        <child link="lower_arm_link" />
+        <axis xyz="0 0 1" />
+        <limit upper="${pi/2}" lower="-${pi/2}" effort="1.0" velocity="1.0" />
+    </joint>
+    <link name="wrist_link">
+        <visual>
+            <origin xyz="0 0 0" rpy="-${pi/2} ${pi/2} 0" />
+            <geometry>
+                <mesh filename="package://my_arm_description/meshes/Wrist_Pitch_Roll.STL" />
+            </geometry>
+        </visual>
+    </link>
+    <joint name="lower_arm_to_wrist_joint" type="revolute">
+        <origin xyz="0.135 0.0052 0.0" rpy="0 0 0" />
+        <parent link="lower_arm_link" />
+        <child link="wrist_link" />
+        <axis xyz="0 0 1" />
+        <limit upper="${pi/2}" lower="-${pi/2}" effort="1.0" velocity="1.0" />
+    </joint>
+    <link name="fixed_jaw_link">
+        <visual>
+            <origin xyz="0 0 0" rpy="-${pi/2} 0 -${pi/2}" />
+            <geometry>
+                <mesh filename="package://my_arm_description/meshes/Fixed_Jaw.STL" />
+            </geometry>
+        </visual>
+    </link>
+    <joint name="wrist_to_fixed_jaw_joint" type="revolute">
+        <origin xyz="0.06 0.0 0.0" rpy="0 ${pi/2} 0" />
+        <parent link="wrist_link" />
+        <child link="fixed_jaw_link" />
+        <axis xyz="0 0 1" />
+        <limit upper="${pi}" lower="-${pi}" effort="1.0" velocity="1.0" />
+    </joint>
+    <link name="moving_jaw_link">
+        <visual>
+            <origin xyz="0 0 0" rpy="0 0 0" />
+            <geometry>
+                <mesh filename="package://my_arm_description/meshes/Moving_Jaw.STL" />
+            </geometry>
+        </visual>
+    </link>
+    <joint name="fixed_to_moving_jaw_joint" type="revolute">
+        <origin xyz="0.0 0.02 0.0245" rpy="${pi/2} ${pi} -${pi/2}" />
+        <parent link="fixed_jaw_link" />
+        <child link="moving_jaw_link" />
+        <axis xyz="0 0 1" />
+        <limit upper="${pi/2}" lower="-${pi/2}" effort="1.0" velocity="1.0" />
     </joint>
 </robot>

Commit message: Launch file to spawn SOARM100 in a custom world
- update `src/my_worlds/README.md` - add notes on issues with paths
  and environmental variables

- in `src/my_arm_description`:
  - in `CMakeLists.txt` - install `launch` folder
  - in `urdf/my_arm.urdf.xacro` - add <collision> and <inertial>
    for all links and adjust upper/lower limits for joints
  - new `launch/my_arm.launch.py` launch file - spawn SOARM100
    robot arm in `duckieworld.sdf` world with `greentable`, several
    `whitecubes`, a `duckie` and a `barrel`

File: src/my_arm_description/urdf/my_arm.urdf.xacro (robot description, xacro)
@@ -9,4 +9,17 @@
             </geometry>
         </visual>
+        <collision>
+            <origin xyz="0 0 0" rpy="0 0 0" />
+            <geometry>
+                <mesh filename="package://my_arm_description/meshes/Base.STL" />
+            </geometry>
+        </collision>
+        <inertial>
+            <mass value="0.1" />
+            <origin xyz="0 0 0" rpy="0 0 0" />
+            <inertia ixx="0.001" ixy="0.0" ixz="0.0"
+                iyy="0.001" iyz="0.0"
+                izz="0.001" />
+        </inertial>
     </link>
     <joint name="world_to_base_joint" type="fixed">
@@ -22,4 +35,17 @@
             </geometry>
         </visual>
+        <collision>
+            <origin xyz="0 0 0" rpy="${pi/2} 0 0" />
+            <geometry>
+                <mesh filename="package://my_arm_description/meshes/Rotation_Pitch.STL" />
+            </geometry>
+        </collision>
+        <inertial>
+            <mass value="0.1" />
+            <origin xyz="0 0 0" rpy="0 0 0" />
+            <inertia ixx="0.001" ixy="0.0" ixz="0.0"
+                iyy="0.001" iyz="0.0"
+                izz="0.001" />
+        </inertial>
     </link>
     <joint name="base_to_shoulder_joint" type="revolute">
@@ -28,5 +54,5 @@
         <child link="shoulder_link" />
         <axis xyz="0 0 1" />
-        <limit upper="${pi/2}" lower="-${pi/2}" effort="1.0" velocity="1.0" />
+        <limit upper="${2*pi/3}" lower="-${2*pi/3}" effort="1.0" velocity="1.0" />
     </joint>
     <link name="upper_arm_link">
@@ -37,4 +63,17 @@
             </geometry>
         </visual>
+        <collision>
+            <origin xyz="0 0 0" rpy="0 ${pi/2} 0" />
+            <geometry>
+                <mesh filename="package://my_arm_description/meshes/Upper_Arm.STL" />
+            </geometry>
+        </collision>
+        <inertial>
+            <mass value="0.1" />
+            <origin xyz="0 0 0" rpy="0 0 0" />
+            <inertia ixx="0.001" ixy="0.0" ixz="0.0"
+                iyy="0.001" iyz="0.0"
+                izz="0.001" />
+        </inertial>
     </link>
     <joint name="shoulder_to_upper_arm_joint" type="revolute">
@@ -43,5 +82,5 @@
         <child link="upper_arm_link" />
         <axis xyz="0 0 1" />
-        <limit upper="${pi/2}" lower="-${pi/2}" effort="1.0" velocity="1.0" />
+        <limit upper="${2*pi/3}" lower="-${2*pi/3}" effort="1.0" velocity="1.0" />
     </joint>
     <link name="lower_arm_link">
@@ -52,4 +91,17 @@
             </geometry>
         </visual>
+        <collision>
+            <origin xyz="0 0 0" rpy="0 ${pi/2} 0" />
+            <geometry>
+                <mesh filename="package://my_arm_description/meshes/Lower_Arm.STL" />
+            </geometry>
+        </collision>
+        <inertial>
+            <mass value="0.1" />
+            <origin xyz="0 0 0" rpy="0 0 0" />
+            <inertia ixx="0.001" ixy="0.0" ixz="0.0"
+                iyy="0.001" iyz="0.0"
+                izz="0.001" />
+        </inertial>
     </link>
     <joint name="upper_arm_to_lower_arm_joint" type="revolute">
@@ -67,4 +119,17 @@
             </geometry>
         </visual>
+        <collision>
+            <origin xyz="0 0 0" rpy="-${pi/2} ${pi/2} 0" />
+            <geometry>
+                <mesh filename="package://my_arm_description/meshes/Wrist_Pitch_Roll.STL" />
+            </geometry>
+        </collision>
+        <inertial>
+            <mass value="0.1" />
+            <origin xyz="0 0 0" rpy="0 0 0" />
+            <inertia ixx="0.001" ixy="0.0" ixz="0.0"
+                iyy="0.001" iyz="0.0"
+                izz="0.001" />
+        </inertial>
     </link>
     <joint name="lower_arm_to_wrist_joint" type="revolute">
@@ -73,5 +138,5 @@
         <child link="wrist_link" />
         <axis xyz="0 0 1" />
-        <limit upper="${pi/2}" lower="-${pi/2}" effort="1.0" velocity="1.0" />
+        <limit upper="${2*pi/3}" lower="-${2*pi/3}" effort="1.0" velocity="1.0" />
     </joint>
     <link name="fixed_jaw_link">
@@ -82,4 +147,17 @@
             </geometry>
         </visual>
+        <collision>
+            <origin xyz="0 0 0" rpy="-${pi/2} 0 -${pi/2}" />
+            <geometry>
+                <mesh filename="package://my_arm_description/meshes/Fixed_Jaw.STL" />
+            </geometry>
+        </collision>
+        <inertial>
+            <mass value="0.1" />
+            <origin xyz="0 0 0" rpy="0 0 0" />
+            <inertia ixx="0.001" ixy="0.0" ixz="0.0"
+                iyy="0.001" iyz="0.0"
+                izz="0.001" />
+        </inertial>
     </link>
     <joint name="wrist_to_fixed_jaw_joint" type="revolute">
@@ -88,5 +166,5 @@
         <child link="fixed_jaw_link" />
         <axis xyz="0 0 1" />
-        <limit upper="${pi}" lower="-${pi}" effort="1.0" velocity="1.0" />
+        <limit upper="${7*pi/6}" lower="-${7*pi/6}" effort="1.0" velocity="1.0" />
     </joint>
     <link name="moving_jaw_link">
@@ -97,4 +175,17 @@
             </geometry>
         </visual>
+        <collision>
+            <origin xyz="0 0 0" rpy="0 0 0" />
+            <geometry>
+                <mesh filename="package://my_arm_description/meshes/Moving_Jaw.STL" />
+            </geometry>
+        </collision>
+        <inertial>
+            <mass value="0.1" />
+            <origin xyz="0 0 0" rpy="0 0 0" />
+            <inertia ixx="0.001" ixy="0.0" ixz="0.0"
+                iyy="0.001" iyz="0.0"
+                izz="0.001" />
+        </inertial>
     </link>
     <joint name="fixed_to_moving_jaw_joint" type="revolute">
@@ -103,5 +194,5 @@
         <child link="moving_jaw_link" />
         <axis xyz="0 0 1" />
-        <limit upper="${pi/2}" lower="-${pi/2}" effort="1.0" velocity="1.0" />
+        <limit upper="${2*pi/3}" lower="-${pi/6}" effort="1.0" velocity="1.0" />
     </joint>
 </robot>

Commit message: Launch RVIZ and Joint State Publisher GUI, fix visuals
- in `src/my_arm_description/`:
   - in `launch/my_arm.launch.py` - launch RVIZ and
     Joint State Publisher GUI
   - `urdf/my_arm.urdf.xacro` - add materials to <visual> tags of
     <links> of the robot to fix display (was white in Gazebo and
     red in RVIZ)
   - new `/config/my_arm.rviz` - RVIZ config file with defaults for
     visualization and panels
   - in `CMakeLists.txt` - install new `config/` folder

File: src/my_arm_description/urdf/my_arm.urdf.xacro (robot description, xacro)
@@ -1,4 +1,9 @@
 <?xml version="1.0" encoding="utf-8"?>
 <robot xmlns:xacro="http://www.ros.org/wiki/xacro" name="my_arm">
+    <xacro:macro name="colored_material" params="name rgba">
+        <material name="${name}">
+            <color rgba="${rgba}" />
+        </material>
+    </xacro:macro>
     <link name="world" />
     <link name="base_link">
@@ -8,4 +13,5 @@
                 <mesh filename="package://my_arm_description/meshes/Base.STL" />
             </geometry>
+            <xacro:colored_material name="White" rgba=".9 .9 .9 .9" />
         </visual>
         <collision>
@@ -34,4 +40,5 @@
                 <mesh filename="package://my_arm_description/meshes/Rotation_Pitch.STL" />
             </geometry>
+            <xacro:colored_material name="White" rgba=".9 .9 .9 .9" />
         </visual>
         <collision>
@@ -62,4 +69,5 @@
                 <mesh filename="package://my_arm_description/meshes/Upper_Arm.STL" />
             </geometry>
+            <xacro:colored_material name="White" rgba=".9 .9 .9 .9" />
         </visual>
         <collision>
@@ -90,4 +98,5 @@
                 <mesh filename="package://my_arm_description/meshes/Lower_Arm.STL" />
             </geometry>
+            <xacro:colored_material name="White" rgba=".9 .9 .9 .9" />
         </visual>
         <collision>
@@ -118,4 +127,5 @@
                 <mesh filename="package://my_arm_description/meshes/Wrist_Pitch_Roll.STL" />
             </geometry>
+            <xacro:colored_material name="White" rgba=".9 .9 .9 .9" />
         </visual>
         <collision>
@@ -146,4 +156,5 @@
                 <mesh filename="package://my_arm_description/meshes/Fixed_Jaw.STL" />
             </geometry>
+            <xacro:colored_material name="White" rgba=".9 .9 .9 .9" />
         </visual>
         <collision>
@@ -174,4 +185,5 @@
                 <mesh filename="package://my_arm_description/meshes/Moving_Jaw.STL" />
             </geometry>
+            <xacro:colored_material name="White" rgba=".9 .9 .9 .9" />
         </visual>
         <collision>

Commit message: Add ros2_control support (WIP)
Not working yet: it complains gz_ros2_control shared library not found

- in `src/my_arm_description/`:
   - in `launch/my_arm.launch.py` - launch ros2_control
   - in `urdf/my_arm.urdf.xacro` - add ros2_control support
   - new `README.md` - notes on adding ros2_control support
      - new `/config/ros2_controllers.yaml` - parameter file for the
        controller manager

File: src/my_arm_description/urdf/my_arm.urdf.xacro (robot description, xacro)
@@ -208,3 +208,32 @@
         <limit upper="${2*pi/3}" lower="-${pi/6}" effort="1.0" velocity="1.0" />
     </joint>
+    <!-- ros2_control -->
+    <xacro:macro name="ros2_position_controller" params="joint_name">
+        <joint name="${joint_name}">
+            <command_interface name="position" />
+            <state_interface name="position">
+                <param name="initial_value">0.0</param>
+            </state_interface>
+            <state_interface name="velocity" />
+        </joint>
+    </xacro:macro>
+    <ros2_control name="my_arm" type="system">
+        <hardware>
+            <plugin>gz_ros2_control/GazeboSimSystem</plugin>
+        </hardware>
+        <xacro:ros2_position_controller joint_name="base_to_shoulder_joint" />
+        <xacro:ros2_position_controller joint_name="shoulder_to_upper_arm_joint" />
+        <xacro:ros2_position_controller joint_name="upper_arm_to_lower_arm_joint" />
+        <xacro:ros2_position_controller joint_name="lower_arm_to_wrist_joint" />
+        <xacro:ros2_position_controller joint_name="wrist_to_fixed_jaw_joint" />
+        <xacro:ros2_position_controller joint_name="fixed_to_moving_jaw_joint" />
+    </ros2_control>
+    <gazebo>
+        <plugin filename="gz_ros2_control-system" name="gz_ros2_control::GazeboSimROS2ControlPlugin">
+            <parameters>$(find my_arm_description)/config/ros2_controllers.yaml</parameters>
+        </plugin>
+        <plugin filename="gz-sim-sensors-system" name="gz::sim::systems::Sensors">
+            <render_engine>ogre2</render_engine>
+        </plugin>
+    </gazebo>
 </robot>

Commit message: Add camera and parametrize robot color

File: src/my_arm_description/urdf/my_arm.urdf.xacro (robot description, xacro)
@@ -1,9 +1,7 @@
 <?xml version="1.0" encoding="utf-8"?>
 <robot xmlns:xacro="http://www.ros.org/wiki/xacro" name="my_arm">
-    <xacro:macro name="colored_material" params="name rgba">
-        <material name="${name}">
-            <color rgba="${rgba}" />
-        </material>
-    </xacro:macro>
+    <material name="robot_color">
+        <color rgba="0.9 0.9 0.9 0.9" />
+    </material>
     <link name="world" />
     <link name="base_link">
@@ -13,5 +11,5 @@
                 <mesh filename="package://my_arm_description/meshes/Base.STL" />
             </geometry>
-            <xacro:colored_material name="White" rgba=".9 .9 .9 .9" />
+            <material name="robot_color"/>
         </visual>
         <collision>
@@ -40,5 +38,5 @@
                 <mesh filename="package://my_arm_description/meshes/Rotation_Pitch.STL" />
             </geometry>
-            <xacro:colored_material name="White" rgba=".9 .9 .9 .9" />
+            <material name="robot_color"/>
         </visual>
         <collision>
@@ -69,5 +67,5 @@
                 <mesh filename="package://my_arm_description/meshes/Upper_Arm.STL" />
             </geometry>
-            <xacro:colored_material name="White" rgba=".9 .9 .9 .9" />
+            <material name="robot_color"/>
         </visual>
         <collision>
@@ -98,5 +96,5 @@
                 <mesh filename="package://my_arm_description/meshes/Lower_Arm.STL" />
             </geometry>
-            <xacro:colored_material name="White" rgba=".9 .9 .9 .9" />
+            <material name="robot_color"/>
         </visual>
         <collision>
@@ -127,5 +125,5 @@
                 <mesh filename="package://my_arm_description/meshes/Wrist_Pitch_Roll.STL" />
             </geometry>
-            <xacro:colored_material name="White" rgba=".9 .9 .9 .9" />
+            <material name="robot_color"/>
         </visual>
         <collision>
@@ -156,5 +154,5 @@
                 <mesh filename="package://my_arm_description/meshes/Fixed_Jaw.STL" />
             </geometry>
-            <xacro:colored_material name="White" rgba=".9 .9 .9 .9" />
+            <material name="robot_color"/>
         </visual>
         <collision>
@@ -185,5 +183,5 @@
                 <mesh filename="package://my_arm_description/meshes/Moving_Jaw.STL" />
             </geometry>
-            <xacro:colored_material name="White" rgba=".9 .9 .9 .9" />
+            <material name="robot_color"/>
         </visual>
         <collision>
@@ -208,4 +206,9 @@
         <limit upper="${2*pi/3}" lower="-${pi/6}" effort="1.0" velocity="1.0" />
     </joint>
+    <!-- Include camera -->
+    <xacro:include filename="$(find my_arm_description)/urdf/my_camera.xacro" />
+    <xacro:camera world_link_name="world">
+        <origin xyz="0 0.2 .2" rpy="0 0 ${-pi/2}" />
+    </xacro:camera>
     <!-- ros2_control -->
     <xacro:macro name="ros2_position_controller" params="joint_name">
