Commit message: Parametrize my_camera.xacro to enable multiple cameras
- in `urdf/my_camera.xacro` add a `camera_name` parameter to xacro:macro "camera"
  to produce customized topics, links and joints in order to enable spawning
  multiple cameras

- in `urdf/my_arm.urdf.xacro` modify call to xacro:macro camera to spawn
  wrist_camera linked to fixed_jaw_link in correct position

- in `launch/my_arm.launch.py` use custom topics in calls to ros_gz_bridge and
  image_bridge

File: src/my_arm_description/urdf/my_arm.urdf.xacro (robot description, xacro)
@@ -206,9 +206,15 @@
         <limit upper="${2*pi/3}" lower="-${pi/6}" effort="1.0" velocity="1.0" />
     </joint>
-    <!-- Include camera -->
+    <!-- Include cameras -->
     <xacro:include filename="$(find my_arm_description)/urdf/my_camera.xacro" />
-    <xacro:camera world_link_name="world">
-        <origin xyz="0 0.2 .2" rpy="0 0 ${-pi/2}" />
+    <xacro:camera world_link_name="fixed_jaw_link" camera_name="wrist_camera">
+        <!--origin xyz="-0.02 0.0 0.05" rpy="0 0.4 ${-pi/2}" /-->
+        <origin xyz="-0.05 0.0 0.01" rpy="0 ${-pi/2+0.4} 0 " />
     </xacro:camera>
+    <!--
+    <xacro:camera world_link_name="world" camera_name="tripod_camera">
+        <origin xyz="0.2 0.2 .2" rpy="0 0 ${-pi/3}" />
+    </xacro:camera>
+    -->
     <!-- ros2_control -->
     <xacro:macro name="ros2_position_controller" params="joint_name">

File: src/my_arm_description/urdf/my_camera.xacro (robot description, xacro)
@@ -2,11 +2,11 @@
 <robot name="my_camera"
     xmlns:xacro="http://ros.org/wiki/xacro">
-    <xacro:macro name="camera" params="world_link_name *origin">
+    <xacro:macro name="camera" params="camera_name world_link_name *origin">
         <!-- Define the material once -->
         <material name="orange">
             <color rgba="1.0 0.55 0.0 1.0" />
         </material>
-        <!-- Fixed Camera Link -->
-        <link name="camera_link">
+        <!-- Camera Link -->
+        <link name="${camera_name}_link">
             <visual>
                 <geometry>
@@ -28,18 +28,18 @@
             </inertial>
         </link>
-        <joint name="camera_optical_joint" type="fixed">
-            <parent link="camera_link" />
-            <child link="camera_link_optical" />
+        <joint name="${camera_name}_optical_joint" type="fixed">
+            <parent link="${camera_name}_link" />
+            <child link="${camera_name}_link_optical" />
             <origin xyz="0 0 0" rpy="${-pi/2} 0 ${-pi/2}" />
         </joint>
-        <link name="camera_link_optical"></link>
-        <gazebo reference="camera_link">
+        <link name="${camera_name}_link_optical"></link>
+        <gazebo reference="${camera_name}_link">
             <material>Gazebo/Orange</material>
-            <sensor type="camera" name="camera_sensor">
+            <sensor type="camera" name="${camera_name}_sensor">
                 <always_on>true</always_on>
                 <update_rate>30.0</update_rate>
                 <visualize>true</visualize>
                 <camera>
-                    <camera_info>camera/camera_info</camera_info>
+                    <camera_info>${camera_name}/camera_info</camera_info>
                     <horizontal_fov>1.047</horizontal_fov> <!-- ~60 degrees UPDATE THESE VALUES-->
                     <image>
@@ -49,15 +49,15 @@
                     </image>
                     <clip>
-                        <near>0.1</near>
+                        <near>0.01</near>
                         <far>20.0</far>
                     </clip>
                 </camera>
-                <topic>camera/image_raw</topic>
-                <gz_frame_id>camera_link_optical</gz_frame_id>
+                <topic>${camera_name}/image_raw</topic>
+                <gz_frame_id>${camera_name}_link_optical</gz_frame_id>
             </sensor>
         </gazebo>
         <!-- Joint from world to camera_link -->
-        <joint name="camera_to_world_joint" type="fixed">
-            <child link="camera_link" />
+        <joint name="${camera_name}_to_parent_joint" type="fixed">
+            <child link="${camera_name}_link" />
             <parent link="${world_link_name}" />
             <xacro:insert_block name="origin" />

Commit message: Add wrist camera mount
 * in `CAD/` folder rename and reorder files in folders. Create new
   folder `v3_export_to_gazebo` - scale down `my_wrist_camera_mount_v3`
   x1000 to transform units from mm to m, place it in position relative
   to `Fixed_Jaw.STL` and export both files together

 * new `meshes/Fixed_Jaw_w_cam_mount_v3.STL` - STL export from
   `fixed_jaw_with_wrist_camera_mount_v3.FCStd` to load as mesh

 * in `urdf/my_arm.urdf.xacro`:
   * load `Fixed_Jaw_w_cam_mount_v3.STL` instead of `Fixed_Jaw.STL`
     mesh both in <visual> and <collision>
   * adjust origin to properly align camera with mount:
-        <origin xyz="-0.05 0.0 0.01" rpy="0 ${-pi/2+0.4} 0 " />
+        <origin xyz="-0.082 0.002 0.044" rpy="0 ${-pi/2+0.95} 0 " />

   * import realsense (not working yet):

* in `urdf/my_camera.xacro ` - modify camera dimensions and colors
  to be more realistic

File: src/my_arm_description/urdf/my_arm.urdf.xacro (robot description, xacro)
@@ -152,5 +152,5 @@
             <origin xyz="0 0 0" rpy="-${pi/2} 0 -${pi/2}" />
             <geometry>
-                <mesh filename="package://my_arm_description/meshes/Fixed_Jaw.STL" />
+                <mesh filename="package://my_arm_description/meshes/Fixed_Jaw_w_cam_mount_v3.STL" />
             </geometry>
             <material name="robot_color"/>
@@ -159,5 +159,5 @@
             <origin xyz="0 0 0" rpy="-${pi/2} 0 -${pi/2}" />
             <geometry>
-                <mesh filename="package://my_arm_description/meshes/Fixed_Jaw.STL" />
+                <mesh filename="package://my_arm_description/meshes/Fixed_Jaw_w_cam_mount_v3.STL" />
             </geometry>
         </collision>
@@ -210,5 +210,5 @@
     <xacro:camera world_link_name="fixed_jaw_link" camera_name="wrist_camera">
         <!--origin xyz="-0.02 0.0 0.05" rpy="0 0.4 ${-pi/2}" /-->
-        <origin xyz="-0.05 0.0 0.01" rpy="0 ${-pi/2+0.4} 0 " />
+        <origin xyz="-0.082 0.002 0.044" rpy="0 ${-pi/2+0.95} 0 " />
     </xacro:camera>
     <!--
@@ -217,4 +217,9 @@
     </xacro:camera>
     -->
+    <!-- Import and add realsense -->
+    <xacro:include filename="$(find sensors)/realsense_d435/realsense.urdf.xacro" />
+    <xacro:realsense world_link_name="world">
+        <origin xyz="0 1.00 1.2" rpy="0 ${pi/4} -${pi/2}" />
+    </xacro:realsense>
     <!-- ros2_control -->
     <xacro:macro name="ros2_position_controller" params="joint_name">

File: src/my_arm_description/urdf/my_camera.xacro (robot description, xacro)
@@ -4,6 +4,9 @@
     <xacro:macro name="camera" params="camera_name world_link_name *origin">
         <!-- Define the material once -->
-        <material name="orange">
-            <color rgba="1.0 0.55 0.0 1.0" />
+        <material name="black">
+            <color rgba="0.1 0.1 0.1 1.0" />
+        </material>
+        <material name="green">
+            <color rgba="0.0 0.6 0.2 1.0" />
         </material>
         <!-- Camera Link -->
@@ -11,14 +14,14 @@
             <visual>
                 <geometry>
-                    <box size="0.01 0.03 0.03" />
+                    <box size="0.0015 0.035 0.025" />
                 </geometry>
-                <material name="orange" />
+                <material name="green" />
             </visual>
             <visual>
-                <origin xyz="0 0 -0.05" />
+                <origin xyz="0.0025 0 0" rpy="0 ${pi/2} 0"/>
                 <geometry>
-                    <cylinder radius="0.002" length="0.1" />
+                    <cylinder radius="0.005" length="0.004" />
                 </geometry>
-                <material name="orange" />
+                <material name="black" />
             </visual>
             <inertial>
@@ -35,5 +38,5 @@
         <link name="${camera_name}_link_optical"></link>
         <gazebo reference="${camera_name}_link">
-            <material>Gazebo/Orange</material>
+            <!--material>Gazebo/Orange</material -->
             <sensor type="camera" name="${camera_name}_sensor">
                 <always_on>true</always_on>

Commit message: Fix issue with multiple cameras, display in GUI
 * in `urdf/my_camera.xacro`- move material definition outside of macros to avoid repetition
   this fixes error when spawning multiple cameras

 * in `launch/my_arm.launch.py` - add tripod_camera topics to ros_gz_bridge and image_bridge

 * in `urdf/my_arm.urdf.xacro` - uncomment fixed tripod camera xacro:macro block, adjust
   camera position and orientation
-        <origin xyz="0.2 0.2 .2" rpy="0 0 ${-pi/3}" />
+        <origin xyz="-0.7 0.0 0.5" rpy="0 ${pi/6} -${pi/6}" />

 * in `config/my_arm.rviz` adjust panels to show 2 image displays in RVIZ

 * in `config/gazebo_gui.config` adjust panels to show 2 image displays in Gazebo

File: src/my_arm_description/urdf/my_arm.urdf.xacro (robot description, xacro)
@@ -208,13 +208,12 @@
     <!-- Include cameras -->
     <xacro:include filename="$(find my_arm_description)/urdf/my_camera.xacro" />
+    <!-- Wrist mounted camera -->
     <xacro:camera world_link_name="fixed_jaw_link" camera_name="wrist_camera">
-        <!--origin xyz="-0.02 0.0 0.05" rpy="0 0.4 ${-pi/2}" /-->
         <origin xyz="-0.082 0.002 0.044" rpy="0 ${-pi/2+0.95} 0 " />
     </xacro:camera>
-    <!--
+    <!-- Fixed tripod camera -->
     <xacro:camera world_link_name="world" camera_name="tripod_camera">
-        <origin xyz="0.2 0.2 .2" rpy="0 0 ${-pi/3}" />
+        <origin xyz="-0.7 0.0 0.5" rpy="0 ${pi/6} -${pi/6}" />
     </xacro:camera>
-    -->
     <!-- Import and add realsense -->
     <xacro:include filename="$(find sensors)/realsense_d435/realsense.urdf.xacro" />

File: src/my_arm_description/urdf/my_camera.xacro (robot description, xacro)
@@ -2,12 +2,12 @@
 <robot name="my_camera"
     xmlns:xacro="http://ros.org/wiki/xacro">
-    <xacro:macro name="camera" params="camera_name world_link_name *origin">
-        <!-- Define the material once -->
-        <material name="black">
+    <!-- Define materials once -->
+        <material name="camera_lens">
             <color rgba="0.1 0.1 0.1 1.0" />
         </material>
-        <material name="green">
+        <material name="PCB">
             <color rgba="0.0 0.6 0.2 1.0" />
         </material>
+    <xacro:macro name="camera" params="camera_name world_link_name *origin">
         <!-- Camera Link -->
         <link name="${camera_name}_link">
@@ -16,5 +16,5 @@
                     <box size="0.0015 0.035 0.025" />
                 </geometry>
-                <material name="green" />
+                <material name="PCB" />
             </visual>
             <visual>
@@ -23,5 +23,5 @@
                     <cylinder radius="0.005" length="0.004" />
                 </geometry>
-                <material name="black" />
+                <material name="camera_lens" />
             </visual>
             <inertial>
